File: hardware/output.kicad_sch (KiCad schematic)
At the start: 10 parts, among them K1 FINDER-30.22, Q2 BSS123, Q3 BSS123

Commit message: working simulations, assigned footprints
"nightly" relase
Parts:
- D3, D4, D5: value 1N5408 -> SK36A; footprint Diode_THT:D_DO-201AD_P15.24mm_Horizontal -> Diode_SMD:D_SMA_Handsoldering
Changed lines of the file:
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@@
       (effects (font (size 1.27 1.27)) (justify left))
     )
-    (property "Value" "1N5408" (id 1) (at 222.25 111.7599 90)
+    (property "Value" "SK36A" (id 1) (at 222.25 111.7599 90)
       (effects (font (size 1.27 1.27)) (justify left))
     )
-    (property "Footprint" "Diode_THT:D_DO-201AD_P15.24mm_Horizontal" (id 2) (at 215.265 110.49 0)
+    (property "Footprint" "Diode_SMD:D_SMA_Handsoldering" (id 2) (at 215.265 110.49 0)
       (effects (font (size 1.27 1.27)) hide)
     )
-    (property "Datasheet" "http://www.vishay.com/docs/88516/1n5400.pdf" (id 3) (at 219.71 110.49 0)
+    (property "Datasheet" "https://www.mouser.pl/datasheet/2/395/SK32A_SERIES_V2102-2822194.pdf" (id 3) (at 219.71 110.49 0)
       (effects (font (size 1.27 1.27)) hide)
     )
@@
       (effects (font (size 1.27 1.27)) (justify left))
     )
-    (property "Value" "1N5408" (id 1) (at 153.67 62.2299 90)
+    (property "Value" "SK36A" (id 1) (at 153.67 62.2299 90)
       (effects (font (size 1.27 1.27)) (justify left))
     )
-    (property "Footprint" "Diode_THT:D_DO-201AD_P15.24mm_Horizontal" (id 2) (at 146.685 60.96 0)
+    (property "Footprint" "Diode_SMD:D_SMA_Handsoldering" (id 2) (at 146.685 60.96 0)
       (effects (font (size 1.27 1.27)) hide)
     )
-    (property "Datasheet" "http://www.vishay.com/docs/88516/1n5400.pdf" (id 3) (at 151.13 60.96 0)
+    (property "Datasheet" "https://www.mouser.pl/datasheet/2/395/SK32A_SERIES_V2102-2822194.pdf" (id 3) (at 151.13 60.96 0)
       (effects (font (size 1.27 1.27)) hide)
     )
@@
       (effects (font (size 1.27 1.27)) (justify left))
     )
-    (property "Value" "1N5408" (id 1) (at 102.87 110.4899 90)
+    (property "Value" "SK36A" (id 1) (at 102.87 110.4899 90)
       (effects (font (size 1.27 1.27)) (justify left))
     )
-    (property "Footprint" "Diode_THT:D_DO-201AD_P15.24mm_Horizontal" (id 2) (at 95.885 109.22 0)
+    (property "Footprint" "Diode_SMD:D_SMA_Handsoldering" (id 2) (at 95.885 109.22 0)
       (effects (font (size 1.27 1.27)) hide)
     )
-    (property "Datasheet" "http://www.vishay.com/docs/88516/1n5400.pdf" (id 3) (at 100.33 109.22 0)
+    (property "Datasheet" "https://www.mouser.pl/datasheet/2/395/SK32A_SERIES_V2102-2822194.pdf" (id 3) (at 100.33 109.22 0)
       (effects (font (size 1.27 1.27)) hide)
     )

Commit message: kończymy balet na dziś
Parts:
- R14, R15, R16, R17: footprint Resistor_SMD:R_0603_1608Metric -> Resistor_SMD:R_0603_1608Metric_Pad0.98x0.95mm_HandSolder
Connections:
- net LINE renamed VALVE_SUPPLY
Other:
- note removed: "LINE means supply connected After LVMS-> ASMS-> RES-> 2 Required by T15 2.2"
Changed lines of the file:
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@@
   (junction (at 101.6 127) (diameter 0) (color 0 0 0 0)
-  )
-  (junction (at 179.07 30.48) (diameter 0) (color 0 0 0 0)
   )
   (junction (at 219.71 128.27) (diameter 0) (color 0 0 0 0)
@@
     (stroke (width 0) (type default) (color 0 0 0 0))
   )
-  (wire (pts (xy 179.07 30.48) (xy 179.07 52.07))
-    (stroke (width 0) (type default) (color 0 0 0 0))
-  )
   (polyline (pts (xy 234.95 113.03) (xy 234.95 118.11))
     (stroke (width 0) (type default) (color 0 0 0 0))
@@
     (stroke (width 0) (type default) (color 0 0 0 0))
   )
-  (wire (pts (xy 179.07 29.21) (xy 179.07 30.48))
-    (stroke (width 0) (type default) (color 0 0 0 0))
-  )
   (wire (pts (xy 116.84 121.92) (xy 116.84 114.3))
     (stroke (width 0) (type default) (color 0 0 0 0))
@@
     (stroke (width 0) (type default) (color 0 0 0 0))
   )
-  (wire (pts (xy 168.91 30.48) (xy 168.91 27.94))
-    (stroke (width 0) (type default) (color 0 0 0 0))
-  )
   (polyline (pts (xy 116.84 114.3) (xy 116.84 114.3))
     (stroke (width 0) (type default) (color 0 0 0 0))
   )
+  (wire (pts (xy 179.07 31.75) (xy 179.07 52.07))
+    (stroke (width 0) (type default) (color 0 0 0 0))
+  )
   (wire (pts (xy 151.13 57.15) (xy 151.13 49.53))
     (stroke (width 0) (type default) (color 0 0 0 0))
@@
   )
   (polyline (pts (xy 113.03 105.41) (xy 113.03 110.49))
-    (stroke (width 0) (type default) (color 0 0 0 0))
-  )
-  (wire (pts (xy 179.07 30.48) (xy 168.91 30.48))
     (stroke (width 0) (type default) (color 0 0 0 0))
   )
@@
   (text "Solenoid low side switches\n" (at 142.24 142.24 0)
     (effects (font (size 2.54 2.54) italic) (justify left bottom))
-  )
-  (text "LINE means supply connected After LVMS-> ASMS-> RES-> 2\nRequired by T15 2.2"
-    (at 195.58 43.18 0)
-    (effects (font (size 1.27 1.27) italic) (justify left bottom))
   )
   (text "fundamental EBS actuator\n" (at 78.74 119.38 0)
@@
     (effects (font (size 1.27 1.27)) (justify right))
   )
+  (hierarchical_label "VALVE_SUPPLY" (shape input) (at 179.07 31.75 90)
+    (effects (font (size 1.27 1.27)) (justify left))
+  )
   (hierarchical_label "VALVE_2_SIG" (shape input) (at 196.85 128.27 180)
     (effects (font (size 1.27 1.27)) (justify right))
   )
-  (symbol (lib_id "power:PWR_FLAG") (at 168.91 27.94 0) (unit 1)
-    (in_bom yes) (on_board yes) (fields_autoplaced)
-    (property "Reference" "#FLG0103" (id 0) (at 168.91 26.035 0)
-      (effects (font (size 1.27 1.27)) hide)
-    )
-    (property "Value" "PWR_FLAG" (id 1) (at 168.91 22.86 0))
-    (property "Footprint" "" (id 2) (at 168.91 27.94 0)
-      (effects (font (size 1.27 1.27)) hide)
-    )
-    (property "Datasheet" "~" (id 3) (at 168.91 27.94 0)
-      (effects (font (size 1.27 1.27)) hide)
-    )
-    (pin "1")
-  )
   (symbol (lib_id "Device:R") (at 219.71 135.89 0) (unit 1)
     (in_bom yes) (on_board yes) (fields_autoplaced)
@@
       (effects (font (size 1.27 1.27)) (justify left))
     )
-    (property "Footprint" "Resistor_SMD:R_0603_1608Metric" (id 2) (at 217.932 135.89 90)
+    (property "Footprint" "Resistor_SMD:R_0603_1608Metric_Pad0.98x0.95mm_HandSolder" (id 2) (at 217.932 135.89 90)
       (effects (font (size 1.27 1.27)) hide)
     )
@@
     )
     (property "Datasheet" "" (id 3) (at 116.84 140.97 0)
-      (effects (font (size 1.27 1.27)) hide)
-    )
-    (pin "1")
-  )
-  (symbol (lib_id "power:LINE") (at 179.07 29.21 0) (unit 1)
-    (in_bom yes) (on_board yes) (fields_autoplaced)
-    (property "Reference" "#PWR032" (id 0) (at 179.07 33.02 0)
-      (effects (font (size 1.27 1.27)) hide)
-    )
-    (property "Value" "LINE" (id 1) (at 179.07 24.13 0))
-    (property "Footprint" "" (id 2) (at 179.07 29.21 0)
-      (effects (font (size 1.27 1.27)) hide)
-    )
-    (property "Datasheet" "" (id 3) (at 179.07 29.21 0)
       (effects (font (size 1.27 1.27)) hide)
     )
@@
     (property "Reference" "R16" (id 0) (at 208.28 134.62 90))
     (property "Value" "1k" (id 1) (at 208.28 132.08 90))
-    (property "Footprint" "Resistor_SMD:R_0603_1608Metric" (id 2) (at 208.28 130.048 90)
+    (property "Footprint" "Resistor_SMD:R_0603_1608Metric_Pad0.98x0.95mm_HandSolder" (id 2) (at 208.28 130.048 90)
       (effects (font (size 1.27 1.27)) hide)
     )
@@
     (property "Reference" "R14" (id 0) (at 90.17 133.35 90))
     (property "Value" "1k" (id 1) (at 90.17 130.81 90))
-    (property "Footprint" "Resistor_SMD:R_0603_1608Metric" (id 2) (at 90.17 128.778 90)
+    (property "Footprint" "Resistor_SMD:R_0603_1608Metric_Pad0.98x0.95mm_HandSolder" (id 2) (at 90.17 128.778 90)
       (effects (font (size 1.27 1.27)) hide)
     )
@@
       (effects (font (size 1.27 1.27)) (justify left))
     )
-    (property "Footprint" "Resistor_SMD:R_0603_1608Metric" (id 2) (at 99.822 134.62 90)
-      (effects (font (size 1.27 1.27)) hide)
-    )
+    (property "Footprint" "Resistor_SMD:R_0603_1608Metric_Pad0.98x0.95mm_HandSolder" (id 2) (at 99.822 134.62 90)
+      (effects (font (size 1.27 1.27)) hide)
+    )
