File: hardware/PUTM_DV_EBS_2023.kicad_pcb (KiCad board)
At the start: 2 copper layers, 100.2 x 50 mm, 98 parts, among them IC1 UCC2946DG4, IC2 SN74LVC1G74DCTR, IC3 SN74LVC1G74DCTR, IC4 ACT4533AYH-T, K1 FINDER-30.22, Q1 BSS123, Q2 BSS123, Q3 BSS123, Q4 BSS123, U1 74157, U5 STM32L4P5RET6, U6 MCP2562-H-SN, Y1 Crystal_GND24

Commit message: minor changes
pre spotkanie comiit ;DD
Parts:
- removed the REF** at (151.8, 98.6)
- added D16: LED, LED_SMD:LED_0603_1608Metric, F.Cu at (144.7, 85.1)
- added D17: LED, LED_SMD:LED_0603_1608Metric, F.Cu at (155.1, 74.1)
- added D18: LED, LED_SMD:LED_0603_1608Metric, F.Cu at (149.2, 78.8)
- added J2: Conn_01x05, Connector_PinHeader_2.54mm:PinHeader_1x05_P2.54mm_Vertical, F.Cu at (220.1, 38.3)
- added K2: FINDER-30.22, Relay_THT:Relay_DPDT_Finder_30.22, F.Cu at (261.4, 98.7)
- added R2: 2.2k, Resistor_SMD:R_0603_1608Metric, F.Cu at (153.2, 78.8)
- added R34: 2.2k, Resistor_SMD:R_0603_1608Metric, F.Cu at (159.9, 69.1)
- added R35: 2.2k, Resistor_SMD:R_0603_1608Metric, F.Cu at (164.2, 66.5)
- added R36: 2.2k, Resistor_SMD:R_0603_1608Metric, F.Cu at (159.1, 74.1)
- added R37: 2.2k, Resistor_SMD:R_0603_1608Metric, F.Cu at (148.7, 83.9)
- added R38: 330R 1%, Resistor_SMD:R_0603_1608Metric, F.Cu at (248.0, 44.2)
- added R39: 680R 1%, Resistor_SMD:R_0603_1608Metric, F.Cu at (248.0, 41.6)
- added R4: 2.2k, Resistor_SMD:R_0603_1608Metric, F.Cu at (149.1, 81.4)
- added R40: 1k, Resistor_SMD:R_0603_1608Metric, F.Cu at (253.1, 37.2)
- added R41: 330R 1%, Resistor_SMD:R_0603_1608Metric, F.Cu at (205.3, 66.9)
- added R42: 680R 1%, Resistor_SMD:R_0603_1608Metric, F.Cu at (205.3, 64.4)
- added R43: 1k, Resistor_SMD:R_0603_1608Metric, F.Cu at (210.5, 59.9)
- added R44: 330R 1%, Resistor_SMD:R_0603_1608Metric, F.Cu at (205.3, 83.7)
- added R45: 680R 1%, Resistor_SMD:R_0603_1608Metric, F.Cu at (205.3, 81.2)
- added R46: 1k, Resistor_SMD:R_0603_1608Metric, F.Cu at (210.5, 76.7)
- added R5: 2.2k, Resistor_SMD:R_0603_1608Metric, F.Cu at (159.7, 71.6)
- added U10: MAX4238AUT, Package_TO_SOT_SMD:SOT-23-6, F.Cu at (205.9, 77.7)
- added U2: 4011, Package_SO:TSSOP-14_4.4x5mm_P0.65mm, F.Cu at (134.2, 99.3)
- added U3: 4081, Package_SO:TSSOP-14_4.4x5mm_P0.65mm, F.Cu at (143.0, 92.8)
- added U4: 4071, Package_SO:TSSOP-14_4.4x5mm_P0.65mm, F.Cu at (134.2, 92.8)
- added U7: LM1117-3.3, Package_TO_SOT_SMD:TO-252-3_TabPin2, F.Cu at (135.9, 40.0)
- added U8: MAX4238AUT, Package_TO_SOT_SMD:SOT-23-6, F.Cu at (238.6, 38.6)
- added U9: MAX4238AUT, Package_TO_SOT_SMD:SOT-23-6, F.Cu at (205.9, 60.9)
- C29, C30, C31, C5: value 100nF -> 10nF
- D12, D3, D4, D5: value 1N5408 -> SK36A; footprint Diode_THT:D_DO-201AD_P15.24mm_Horizontal -> Diode_SMD:D_SMA_Handsoldering
- U1: footprint Resistor_SMD:R_0603_1608Metric -> Package_SO:VSSOP-8_2.3x2mm_P0.5mm
- moved K1 135.9 mm to (258.6, 128.1)
- moved Q3 102.4 mm to (204.2, 42.7)
- moved REF** 97.7 mm to (108.3, 150.0)
- moved U1 90.5 mm to (139.2, 104.3)
- moved R8 89.3 mm to (149.1, 101.7)
- moved C2 86.3 mm to (147.4, 103.9)
- moved R7 85.9 mm to (144.0, 106.3)
- moved IC2 85.8 mm to (133.1, 104.9)
- moved C17 82.1 mm to (194.0, 22.6)
- moved Q2 81.5 mm to (209.0, 42.7)
- moved D4 79.4 mm to (206.7, 38.2)
- moved D5 79.4 mm to (184.7, 50.0)
- moved C3 79.2 mm to (154.4, 95.0)
- moved C33 79.2 mm to (151.6, 95.0)
- moved R9 78.9 mm to (144.0, 103.8)
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Connections:
- net /EBS Logic/WATCHDOG uC FAULT LATCH renamed /EBS Logic/RESET BUTTON LATCH
- U1 pad 1: /EBS Logic/AS_DRIVING_MODE -> /EBS Logic/TS_ON_COCKPIT
- U1 pad 2: /EBS Logic/TS_ON_COCKPIT -> /EBS Logic/TS_ON_EXT
- U5 pad 10: unconnected-(U5-Pad10) -> /Air pressure sensor control/MAIN
- U5 pad 14: unconnected-(U5-Pad14) -> /EBS Supervisor/OK
- U5 pad 15: unconnected-(U5-Pad15) -> /EBS Supervisor/WARNING
- U5 pad 16: unconnected-(U5-Pad16) -> /EBS Supervisor/ERROR
- U5 pad 21: /EBS Logic/WATCHDOG -> Net-(R4-Pad1)
- U5 pad 22: /EBS Logic/AS_CLOSE_SDC -> Net-(R5-Pad1)
- U5 pad 23: /EBS Logic/AS_DRIVING_MODE -> Net-(R34-Pad1)
- U5 pad 26: unconnected-(U5-Pad26) -> AUX1
- U5 pad 27: unconnected-(U5-Pad27) -> AUX2
- U5 pad 38: /EBS Logic/SDC READY -> Net-(R2-Pad2)
- U5 pad 8: unconnected-(U5-Pad8) -> /Air pressure sensor control/REDUNDANT
- U5 pad 9: unconnected-(U5-Pad9) -> /Air pressure sensor control/EBS
Routing:
- net GND: track 7.56 -> 0.00 mm

Commit message: kończymy balet na dziś
Parts:
- removed D6: D_Schottky, Diode_SMD:D_SMB
- added C34: 5.6n, Capacitor_SMD:C_0603_1608Metric, F.Cu at (224.8, 61.6)
- added C35: 5.6n, Capacitor_SMD:C_0603_1608Metric, F.Cu at (174.1, 98.8)
- added C36: 5.6n, Capacitor_SMD:C_0603_1608Metric, F.Cu at (264.1, 36.7)
- added D2: PESD2CAN.215, Package_TO_SOT_SMD:SOT-23, F.Cu at (204.5, 33.0)
- added J1: SAFETY_SUPPLY, PUTM_Kicad_FOOTPRINTS:M80-5L104YYMC, F.Cu at (139.3, 44.7)
- added J3: SENSORS, PUTM_Kicad_FOOTPRINTS:M80-5L104YYMC, F.Cu at (156.8, 44.7)
- added J4: VALVES, PUTM_Kicad_FOOTPRINTS:M80-5L104YYMC, F.Cu at (164.8, 32.9)
- added J5: MAIN, PUTM_Kicad_FOOTPRINTS:M80-5L112YYMC, F.Cu at (147.3, 32.9)
- C1, C2, C3, C4, C5, C6: footprint Capacitor_SMD:C_0201_0603Metric_Pad0.64x0.40mm_HandSolder -> Capacitor_SMD:C_0603_1608Metric_Pad1.08x0.95mm_HandSolder
- C16, C19, C20: footprint Capacitor_SMD:C_1206_3216Metric -> Capacitor_SMD:C_0603_1608Metric_Pad1.08x0.95mm_HandSolder
- C18: footprint Capacitor_SMD:C_1206_3216Metric -> Capacitor_SMD:C_0805_2012Metric_Pad1.18x1.45mm_HandSolder
- D10: value D_Zener -> BZX38450-C3V3-QX
- D11, D8: footprint LED_SMD:LED_PLCC-2 -> LED_SMD:LED_0603_1608Metric_Pad1.05x0.95mm_HandSolder
- D16, D17, D18: footprint LED_SMD:LED_0603_1608Metric -> LED_SMD:LED_0603_1608Metric_Pad1.05x0.95mm_HandSolder
- J2: value Conn_01x05 -> SWDIO_CONN
- L2: value 47uH TDK -> 47uH; footprint Inductor_SMD:L_1210_3225Metric -> PUTM_Kicad_FOOTPRINTS:L_Bourns_SRP1038WA
- R1, R10, R11, R14, R15, R16, R17, R18, R2, R20, R21, R22, R23, R24, R25, R27, R28, R29, R3, R30, R31, R32, R33, R34, R35, R36, R37, R4, R40, R43, R46, R5, R6, R7, R8, R9: footprint Resistor_SMD:R_0603_1608Metric -> Resistor_SMD:R_0603_1608Metric_Pad0.98x0.95mm_HandSolder
- R38, R41, R44: value 330R 1% -> 3.3k 1%; footprint Resistor_SMD:R_0603_1608Metric -> Resistor_SMD:R_0603_1608Metric_Pad0.98x0.95mm_HandSolder
- R39, R42, R45: value 680R 1% -> 6.8k 1%; footprint Resistor_SMD:R_0603_1608Metric -> Resistor_SMD:R_0603_1608Metric_Pad0.98x0.95mm_HandSolder
- U10, U8, U9: value MAX4238AUT -> TSX7191; footprint Package_TO_SOT_SMD:SOT-23-6 -> Package_TO_SOT_SMD:SOT-23-5_HandSoldering
- moved K1 129.4 mm to (131.8, 102.5)
- moved C10 90.2 mm to (213.5, 32.1)
- moved R10 89.4 mm to (253.1, 68.7)
- moved C5 84.9 mm to (248.1, 71.6)
- moved C7 83.9 mm to (217.8, 32.1)
- moved D1 83.6 mm to (248.4, 68.9)
- moved C9 78.9 mm to (217.8, 34.6)
- moved R11 77.5 mm to (248.1, 74.1)
- moved D16 76.8 mm to (204.3, 36.6)
- moved Q2 75.8 mm to (158.9, 99.7)
- moved Q3 75.8 mm to (154.0, 99.7)
- moved D3 75.8 mm to (144.7, 106.9)
- moved D4 75.8 mm to (156.6, 95.2)
- moved D5 75.8 mm to (134.6, 106.9)
- moved R17 75.7 mm to (131.8, 110.5)
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Connections:
- F1 pad 1: Net-(D6-Pad2) -> /Power Supply/critical_C
- K1 pad 14: LINE -> /Safety Relay/VALVE_SUPPLY
- K2 pad 21: unconnected-(K2-Pad21) -> /Safety Relay/VALVE_SUPPLY
- K2 pad 24: unconnected-(K2-Pad24) -> LINE
- R38 pad 2: Net-(R38-Pad2) -> Net-(R39-Pad1)
- R39 pad 1: Net-(R38-Pad2) -> Net-(R39-Pad1)
- R41 pad 2: Net-(R41-Pad2) -> Net-(R42-Pad1)
- R42 pad 1: Net-(R41-Pad2) -> Net-(R42-Pad1)
- R44 pad 2: Net-(R44-Pad2) -> Net-(R45-Pad1)
- R45 pad 1: Net-(R44-Pad2) -> Net-(R45-Pad1)
- U10 pad 1: Net-(R46-Pad1) -> Net-(R45-Pad1)
- U10 pad 2: GND -> Net-(R46-Pad1)
- U10 pad 3: Net-(R44-Pad2) -> Net-(R46-Pad1)
- U10 pad 4: Net-(R46-Pad1) -> +5V
- U10 pad 5: +5V -> GND
- U8 pad 1: Net-(R40-Pad1) -> Net-(R39-Pad1)
- U8 pad 2: GND -> Net-(R40-Pad1)
- U8 pad 3: Net-(R38-Pad2) -> Net-(R40-Pad1)
- U8 pad 4: Net-(R40-Pad1) -> +5V
- U8 pad 5: +5V -> GND
- U9 pad 1: Net-(R43-Pad1) -> Net-(R42-Pad1)
- U9 pad 2: GND -> Net-(R43-Pad1)
- U9 pad 3: Net-(R41-Pad2) -> Net-(R43-Pad1)
- U9 pad 4: Net-(R43-Pad1) -> +5V
- U9 pad 5: +5V -> GND

Commit message: begin of placement process, supply section done
będą obłe ścieżki i chuj
Parts:
- C18: footprint Capacitor_SMD:C_0805_2012Metric_Pad1.18x1.45mm_HandSolder -> Capacitor_SMD:C_1206_3216Metric
- C21, C25, C34, C35, C36: footprint Capacitor_SMD:C_0603_1608Metric -> Capacitor_SMD:C_0603_1608Metric_Pad1.08x0.95mm_HandSolder
- C22, R22, R24: moved to B.Cu
- C24: footprint Capacitor_SMD:C_0603_1608Metric -> Capacitor_SMD:C_0603_1608Metric_Pad1.08x0.95mm_HandSolder; moved to B.Cu
- moved U10 253.8 mm to (14.7, 96.0)
- moved C36 238.3 mm to (32.6, 93.3)
- moved R44 238.3 mm to (28.4, 95.8)
- moved R46 238.3 mm to (34.2, 88.6)
- moved R45 237.5 mm to (28.2, 89.2)
- moved U8 209.0 mm to (14.5, 87.9)
- moved C10 197.9 mm to (28.3, 101.8)
- moved C14 197.9 mm to (19.0, 108.8)
- moved C6 197.9 mm to (23.4, 106.9)
- moved D17 197.9 mm to (23.9, 101.8)
- moved D2 197.9 mm to (19.3, 102.8)
- moved R12 197.9 mm to (28.2, 106.8)
- moved R2 197.9 mm to (23.1, 111.9)
- moved R34 197.9 mm to (23.9, 104.4)
- moved R4 197.9 mm to (18.8, 111.4)
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Connections:
- net /EBS Logic/AS_COMMADNS+WD_OK renamed /EBS Logic/AS_COMMADNS_OK
Routing:
- net GND: vias 0 -> 8

Commit message: JLC fabrication adjustments, assigned nets
sluchajcie historii typ jakis z ryjem do mnie na swiatlach AWF bo pozno ruszylem pozniej sie ustawilismy kolo siebie i go zjadlem na acceleration new beetlem bo ma 110 koni jebaniec pozdrawiam frajera z opla signum
Parts:
- moved R43 171.6 mm to (17.4, 77.8)
- moved F1 97.9 mm to (94.4, 66.3), turned to 90 degrees
- moved U10 57.9 mm to (68.0, 73.4), turned to -90 degrees
- moved R46 39.0 mm to (68.6, 70.2)
- moved R44 37.6 mm to (58.3, 73.0), turned to -90 degrees
- moved U8 36.7 mm to (18.0, 51.4)
- moved R45 35.9 mm to (60.3, 73.0), turned to 90 degrees
- moved C36 32.1 mm to (59.3, 75.6), turned to 180 degrees
- moved U9 5.67 mm to (17.6, 85.0), turned to -90 degrees
- moved REF** 4.46 mm to (37.5, 167.8)
- moved C35 4.34 mm to (189.4, 100.6)
- moved D7 3.17 mm to (99.4, 66.3)
- moved C16 0.24 mm to (96.4, 155.8)
- moved J4 0.15 mm to (114.4, 62.2)
Routing:
- added copper zone on F.Cu, net Net-(R46-Pad1)
Other:
- copper layers 2 -> 4
- rule pad_to_mask_clearance: 0 -> 0.05

Commit message: dobra ide spać
Parts:
- added REF**: MountingHole_3.2mm_M3_DIN965_Pad_TopBottom, MountingHole:MountingHole_3.2mm_M3_DIN965_Pad_TopBottom, F.Cu at (51.8, 124.2)
- added REF**: MountingHole_3.2mm_M3_DIN965_Pad_TopBottom, MountingHole:MountingHole_3.2mm_M3_DIN965_Pad_TopBottom, F.Cu at (47.0, 68.3)
- added REF**: MountingHole_3.2mm_M3_DIN965_Pad_TopBottom, MountingHole:MountingHole_3.2mm_M3_DIN965_Pad_TopBottom, F.Cu at (134.9, 123.7)
- added REF**: MountingHole_3.2mm_M3_DIN965_Pad_TopBottom, MountingHole:MountingHole_3.2mm_M3_DIN965_Pad_TopBottom, F.Cu at (139.2, 64.3)
- added REF**: WEEE-Logo_5.6x8mm_SilkScreen, Symbol:WEEE-Logo_5.6x8mm_SilkScreen, B.Cu at (99.1, 110.5)
- C18: footprint Capacitor_SMD:C_1206_3216Metric -> Capacitor_SMD:C_0805_2012Metric_Pad1.18x1.45mm_HandSolder
- C21, C24, C25, C34, C35, C36: footprint Capacitor_SMD:C_0603_1608Metric_Pad1.08x0.95mm_HandSolder -> Capacitor_SMD:C_0603_1608Metric
- C23, C27, C28, C29, C30, C31, C32, C33: footprint Capacitor_SMD:C_0201_0603Metric_Pad0.64x0.40mm_HandSolder -> Capacitor_SMD:C_0603_1608Metric_Pad1.08x0.95mm_HandSolder
- G***: moved to F.Cu
- moved R10 217.1 mm to (49.3, 84.1), turned to 180 degrees
- moved C5 211.6 mm to (49.3, 80.8)
- moved R11 211.6 mm to (49.3, 82.4)
- moved R1 203.3 mm to (61.7, 71.9), turned to 180 degrees
- moved R27 190.7 mm to (61.7, 74.5), turned to -90 degrees
- moved R32 182.8 mm to (123.4, 165.1), turned to 180 degrees
- moved R25 178.0 mm to (33.8, 147.8)
- moved R40 168.5 mm to (79.5, 109.7)
- moved D10 168.3 mm to (39.4, 148.1)
- moved C1 168.0 mm to (58.4, 152.3)
- moved C2 168.0 mm to (68.5, 144.2)
- moved C3 168.0 mm to (62.8, 150.2)
- moved C32 168.0 mm to (56.6, 154.9)
- moved C33 168.0 mm to (63.1, 141.0)
- moved C4 168.0 mm to (70.4, 136.7)
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Connections:
- J4 pad 2: VALVE_1_COIL_II -> VALVE_2_COIL_I
- J4 pad 3: VALVE_2_COIL_I -> VALVE_1_COIL_II
Routing:
- net GND: track 0.00 -> 18.4 mm
- net Net-(C35-Pad1): track 0.00 -> 6.29 mm
- net Net-(C34-Pad1): track 0.00 -> 5.65 mm
- net VALVE_1_COIL_I: track 0.00 -> 4.82 mm
- net VALVE_2_COIL_I: track 0.00 -> 4.59 mm
- net Net-(IC4-Pad8): track 0.00 -> 4.50 mm
- net Net-(C36-Pad1): track 0.00 -> 4.43 mm
- net +5V: track 0.00 -> 4.20 mm
- net /EBS Supervisor/XTAL2: track 0.00 -> 4.06 mm
- net /EBS Supervisor/XTAL1: track 0.00 -> 3.69 mm
- net Net-(C22-Pad1): track 0.00 -> 3.61 mm, vias 0 -> 1
- net /Power Supply/critical_C: track 0.00 -> 3.46 mm
- net Net-(IC4-Pad7): track 0.00 -> 3.31 mm, vias 0 -> 1
- net +24V: track 0.00 -> 3.14 mm
- net VALVE_1_COIL_II: track 0.00 -> 3.03 mm
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- added copper zone on F.Cu, net Net-(R40-Pad1)
- added copper zone on F.Cu, net Net-(R43-Pad1)
Other:
- board size 100.2 x 50 mm -> 100 x 70 mm
- board text added: "2nd relay"
- board text added: "ANALOG"
- board text added: "SUPERVISOR"
- board text added: "logic"
- board text removed: "880 213 742"

Commit message: full 3d models, pre-routing, corrections
kurwa bezpiecznik od wczoraj a fura dalej nie jeździ siedze u rakietowcow bo cieplo chlopaki co z wami
Parts:
- removed the REF** at (99.1, 110.5)
- removed the REF** at (69.3, 80.8)
- added H1: MountingHole, MountingHole:MountingHole_3.2mm_M3_ISO7380, F.Cu at (160.3, 111.8)
- added H2: MountingHole, MountingHole:MountingHole_3.2mm_M3_ISO7380, F.Cu at (190.8, 111.8)
- added H3: MountingHole, MountingHole:MountingHole_3.2mm_M3_ISO7380, F.Cu at (160.3, 55.9)
- added H4: MountingHole, MountingHole:MountingHole_3.2mm_M3_ISO7380, F.Cu at (190.8, 55.9)
- added REF**: Cytat, PutRocketLab_graphics:Cytat, B.Cu at (251.9, 106.9)
- C23, C27, C28, C32, C33: footprint Capacitor_SMD:C_0603_1608Metric_Pad1.08x0.95mm_HandSolder -> Capacitor_SMD:C_0201_0603Metric_Pad0.64x0.40mm_HandSolder
- moved G*** 193.6 mm to (273.6, 113.7)
- moved G*** 118.5 mm to (236.0, 119.1)
- moved C31 91.7 mm to (34.5, 139.7)
- moved D15 91.7 mm to (31.8, 142.5)
- moved R32 91.7 mm to (34.5, 142.7)
- moved R33 91.7 mm to (34.5, 141.2)
- moved D10 90.5 mm to (118.6, 104.4)
- moved R25 90.1 mm to (112.8, 104.4)
- moved C10 73.7 mm to (85.4, 148.3)
- moved C14 72.0 mm to (81.3, 144.8)
- moved L1 70.3 mm to (81.6, 157.2)
- moved C6 67.7 mm to (81.3, 142.0)
- moved C12 66.4 mm to (81.3, 148.6)
- moved C7 66.4 mm to (85.5, 142.0)
- moved C9 66.4 mm to (85.5, 144.5)
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Connections:
- D2 pad 1: CAN-L -> CAN+
- D2 pad 2: CAN-H -> CAN-
- J5 pad 1: unconnected-(J5-Pad1) -> CAN-
- J5 pad 10: CAN-H -> AUX1
- J5 pad 11: CAN-L -> unconnected-(J5-Pad11)
- J5 pad 12: unconnected-(J5-Pad12) -> AIR+
- J5 pad 2: TS_ON_EXTERNAL -> DASH_TS_ON
- J5 pad 3: AIR+ -> TS_ON_EXTERNAL
- J5 pad 4: +24V -> unconnected-(J5-Pad4)
- J5 pad 5: GND -> +24V
- J5 pad 6: AUX1 -> GND
- J5 pad 7: EBS_RESET _BUTTON -> CAN+
- J5 pad 8: DASH_TS_ON -> EBS_RESET _BUTTON
- JP1 pad 1: CAN-H -> CAN+
- K1 pad 24: +24V -> /Safety Relay/VALVE_SUPPLY
- R13 pad 2: CAN-L -> CAN-
- U6 pad 6: CAN-L -> CAN-
- U6 pad 7: CAN-H -> CAN+
Routing:
- net AIR+: track 0.00 -> 52.2 mm, vias 0 -> 5
- net VALVE_2_COIL_I: track 4.59 -> 25.4 mm
- net VALVE_1_COIL_I: track 4.82 -> 25.1 mm
- net /Safety Relay/VALVE_SUPPLY: track 0.00 -> 19.8 mm
- net CAN-: track 0.00 -> 8.89 mm
- net CAN+: track 0.00 -> 7.79 mm
- net +24V: track 3.14 -> 9.90 mm
- net Net-(IC1-Pad2): track 0.00 -> 6.43 mm
- net VALVE_2_COIL_II: track 2.98 -> 9.25 mm
- net VALVE_1_COIL_II: track 3.03 -> 9.04 mm
- net Net-(JP1-Pad2): track 0.00 -> 3.49 mm
- net Net-(Q3-Pad1): track 0.00 -> 2.45 mm
- net Net-(C22-Pad1): track 3.61 -> 4.40 mm
- net GND: track 18.4 -> 18.3 mm, vias 8 -> 16
- net /Power Supply/SW_loop: vias 5 -> 4
Other:
- board text added: "Autonomous System Brake"
- board text added: "neighbouring BSPD draft"
- board text added: "relay"
- board text removed: "2nd relay"
- board text removed: "880 299 412"

Commit message: still working
Parts:
- added D6: LED, LED_SMD:LED_0603_1608Metric_Pad1.05x0.95mm_HandSolder, F.Cu at (98.3, 120.7)
- added R47: 2.2k, Resistor_SMD:R_0603_1608Metric_Pad0.98x0.95mm_HandSolder, F.Cu at (98.3, 124.5)
- C29, C30, C31: footprint Capacitor_SMD:C_0603_1608Metric_Pad1.08x0.95mm_HandSolder -> Capacitor_SMD:C_0201_0603Metric_Pad0.64x0.40mm_HandSolder
- moved C32 78.1 mm to (120.2, 101.3), turned to 90 degrees
- moved C15 77.3 mm to (49.0, 83.5), turned to 90 degrees
- moved C4 68.5 mm to (118.7, 107.6), turned to 90 degrees
- moved R6 68.0 mm to (120.0, 110.7)
- moved C28 65.9 mm to (135.1, 104.6), turned to 180 degrees
- moved R7 65.3 mm to (121.2, 105.6), turned to 180 degrees
- moved C33 64.6 mm to (113.4, 101.4), turned to 90 degrees
- moved C23 64.2 mm to (126.8, 104.1), turned to 180 degrees
- moved C14 62.5 mm to (57.4, 87.1)
- moved R3 56.9 mm to (112.9, 116.3), turned to 180 degrees
- moved C27 54.9 mm to (135.2, 117.3), turned to 180 degrees
- moved D17 54.8 mm to (93.5, 120.9), turned to 90 degrees
- moved C10 53.9 mm to (64.0, 98.8), turned to 45 degrees
- moved R16 52.1 mm to (93.2, 107.2), turned to 90 degrees
- moved R36 52.1 mm to (93.5, 124.5), turned to -90 degrees
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Connections:
- D2 pad 1: CAN+ -> CAN-
- D2 pad 2: CAN- -> CAN+
- U5 pad 17: unconnected-(U5-Pad17) -> /EBS Supervisor/CHECKUP
Routing:
- net GND: track 18.3 -> 71.0 mm, vias 16 -> 8
- net /EBS Supervisor/3V3_SYS: track 0.00 -> 8.58 mm
- net CAN+: track 7.79 -> 13.9 mm
- net /EBS Logic/SAFETY_IN: track 0.00 -> 4.01 mm
- net /EBS Logic/TS_ON_EXT: track 0.00 -> 3.76 mm
- net /EBS Logic/TS_ON_COCKPIT: track 0.00 -> 3.66 mm
- net /EBS Logic/SAFETY_RESET_BUT: track 0.00 -> 3.43 mm
- net AIR+: track 52.2 -> 55.2 mm, vias 5 -> 6
- net Net-(Q3-Pad1): track 2.45 -> 0.00 mm
- net +3V3: track 0.00 -> 2.21 mm
- net CAN-: track 8.89 -> 10.9 mm, vias 0 -> 2
- net VALVE_2_COIL_I: track 25.4 -> 23.7 mm
- net VALVE_1_COIL_I: track 25.1 -> 23.6 mm
- net VALVE_2_COIL_II: track 9.25 -> 8.38 mm
- net VALVE_1_COIL_II: track 9.04 -> 8.41 mm
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Other:
- board text added: "LED's"

Commit message: kurde no jeszcze nie skonczylem ale sune dalej
Parts:
- added H1: MountingHole, MountingHole:MountingHole_3.2mm_M3_ISO7380, F.Cu at (22.1, 38.0)
- added H2: MountingHole, MountingHole:MountingHole_3.2mm_M3_ISO7380, F.Cu at (22.1, 68.5)
- added H3: MountingHole, MountingHole:MountingHole_3.2mm_M3_ISO7380, F.Cu at (78.0, 38.0)
- added H4: MountingHole, MountingHole:MountingHole_3.2mm_M3_ISO7380, F.Cu at (78.0, 68.5)
- added REF**: MountingHole_3.2mm_M3_DIN965_Pad_TopBottom, MountingHole:MountingHole_3.2mm_M3_DIN965_Pad_TopBottom, F.Cu at (99.8, 68.8)
- C21, C24, C25, C34, C35, C36: footprint Capacitor_SMD:C_0603_1608Metric -> Capacitor_SMD:C_0603_1608Metric_Pad1.08x0.95mm_HandSolder
- C22: moved to F.Cu
- C27, C28, C29, C30, C31, C32, C33: footprint Capacitor_SMD:C_0201_0603Metric_Pad0.64x0.40mm_HandSolder -> Capacitor_SMD:C_0603_1608Metric_Pad1.08x0.95mm_HandSolder
- D10: footprint Diode_SMD:D_SMB -> Diode_SMD:D_SOD-323_HandSoldering
- R19, R26: footprint Resistor_SMD:R_1206_3216Metric -> Resistor_SMD:R_0603_1608Metric_Pad0.98x0.95mm_HandSolder
- moved G*** 158.6 mm to (123.7, 41.9)
- moved R10 148.0 mm to (151.9, 42.7), turned to -90 degrees
- moved D1 147.4 mm to (148.6, 42.7), turned to 90 degrees
- moved R11 145.7 mm to (150.4, 42.7), turned to 90 degrees
- moved D15 137.2 mm to (168.4, 130.6), turned to 0 degrees
- moved R32 134.9 mm to (168.7, 127.8), turned to -90 degrees
- moved R33 133.3 mm to (167.1, 127.8), turned to 90 degrees
- moved C31 131.6 mm to (165.6, 127.8), turned to 90 degrees
- moved R41 130.5 mm to (103.5, 42.4), turned to 180 degrees
- moved R42 129.9 mm to (103.5, 43.9), turned to 0 degrees
- moved C35 129.3 mm to (103.5, 45.5), turned to 0 degrees
- moved C5 129.2 mm to (170.9, 123.2), turned to -90 degrees
- moved U9 127.8 mm to (103.3, 48.3), turned to 0 degrees
- moved U8 126.1 mm to (111.0, 47.3)
- moved C34 126.1 mm to (113.8, 47.6)
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Connections:
- net /EBS Supervisor/CAN_RX renamed /EBS Supervisor/CAN_RX+
- net /EBS Supervisor/CAN_TX renamed /EBS Supervisor/CAN_TX-
- C17 pad 1: /Power Supply/critical_C -> +24V
- C18 pad 1: /Power Supply/critical_C -> +24V
- D7 pad 1: /Power Supply/critical_C -> +24V
- F1 pad 1: /Power Supply/critical_C -> +24V
- IC4 pad 2: /Power Supply/critical_C -> +24V
Routing:
- net VALVE_2_COIL_I: track 23.7 -> 6.15 mm
- net VALVE_1_COIL_I: track 23.6 -> 6.64 mm
- net CAN-: track 10.9 -> 16.4 mm
- net CAN+: track 13.9 -> 18.9 mm
- net Net-(C22-Pad1): track 4.40 -> 0.00 mm, vias 1 -> 0
- net /EBS Logic/SAFETY_IN: track 4.01 -> 0.02 mm
- net GND: track 71.0 -> 74.9 mm, vias 8 -> 9
- net /Power Supply/critical_C: track 3.46 -> 0.00 mm
- net +24V: track 9.90 -> 13.4 mm
- net Net-(D17-Pad1): track 0.00 -> 1.77 mm
- net Net-(D16-Pad1): track 0.00 -> 1.77 mm
- net Net-(D8-Pad1): track 0.00 -> 1.77 mm
- net Net-(D11-Pad1): track 0.00 -> 1.77 mm
- net Net-(D18-Pad1): track 0.00 -> 1.77 mm
- net /EBS Logic/TS_ON_COCKPIT: track 3.66 -> 5.18 mm
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Other:
- board text added: "3V3"
- board text added: "5V"
- board text added: "CHECKUP"
- board text added: "EBS Logic"
- board text added: "EBS Supervisor"
- board text added: "ERROR"
- board text added: "Input stage"
- board text added: "OK"
- board text added: "Power Supply"
- board text added: "Solenoid Relais"
- board text added: "WARNING"
- board text removed: "ANALOG"
- board text removed: "SUPERVISOR"
- board text removed: "relay"
