File: hardware/supervisor.kicad_sch (KiCad schematic)
At the start: 28 parts, among them U5 STM32L4P5RET6, U6 MCP2562-H-SN, Y1 Crystal_GND24

Commit message: kończymy balet na dziś
Parts:
- C6: footprint Capacitor_SMD:C_0201_0603Metric_Pad0.64x0.40mm_HandSolder -> Capacitor_SMD:C_0603_1608Metric_Pad1.08x0.95mm_HandSolder
- D16, D17, D18: footprint LED_SMD:LED_0603_1608Metric -> LED_SMD:LED_0603_1608Metric_Pad1.05x0.95mm_HandSolder
- D2: footprint (none) -> Package_TO_SOT_SMD:SOT-23
- R2, R34, R35, R36, R37, R4, R5: footprint Resistor_SMD:R_0603_1608Metric -> Resistor_SMD:R_0603_1608Metric_Pad0.98x0.95mm_HandSolder
Changed lines of the file:
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@@
     (property "Reference" "R34" (id 0) (at 153.67 87.63 90))
     (property "Value" "2.2k" (id 1) (at 160.02 88.9 90))
-    (property "Footprint" "Resistor_SMD:R_0603_1608Metric" (id 2) (at 153.67 89.408 90)
+    (property "Footprint" "Resistor_SMD:R_0603_1608Metric_Pad0.98x0.95mm_HandSolder" (id 2) (at 153.67 89.408 90)
       (effects (font (size 1.27 1.27)) hide)
     )
@@
       (effects (font (size 1.27 1.27)) (justify left))
     )
-    (property "Footprint" "" (id 2) (at 255.27 104.14 0)
+    (property "Footprint" "Package_TO_SOT_SMD:SOT-23" (id 2) (at 255.27 104.14 0)
       (effects (font (size 1.27 1.27)) hide)
     )
@@
     (property "Reference" "D16" (id 0) (at 159.0675 62.23 0))
     (property "Value" "LED" (id 1) (at 159.0675 64.77 0))
-    (property "Footprint" "LED_SMD:LED_0603_1608Metric" (id 2) (at 157.48 69.85 0)
+    (property "Footprint" "LED_SMD:LED_0603_1608Metric_Pad1.05x0.95mm_HandSolder" (id 2) (at 157.48 69.85 0)
       (effects (font (size 1.27 1.27)) hide)
     )
@@
     (property "Reference" "D17" (id 0) (at 165.4175 64.77 0))
     (property "Value" "LED" (id 1) (at 165.4175 67.31 0))
-    (property "Footprint" "LED_SMD:LED_0603_1608Metric" (id 2) (at 163.83 72.39 0)
+    (property "Footprint" "LED_SMD:LED_0603_1608Metric_Pad1.05x0.95mm_HandSolder" (id 2) (at 163.83 72.39 0)
       (effects (font (size 1.27 1.27)) hide)
     )
@@
     (property "Reference" "R35" (id 0) (at 182.88 69.85 90))
     (property "Value" "2.2k" (id 1) (at 189.23 71.12 90))
-    (property "Footprint" "Resistor_SMD:R_0603_1608Metric" (id 2) (at 182.88 71.628 90)
+    (property "Footprint" "Resistor_SMD:R_0603_1608Metric_Pad0.98x0.95mm_HandSolder" (id 2) (at 182.88 71.628 90)
       (effects (font (size 1.27 1.27)) hide)
     )
@@
     (property "Reference" "D18" (id 0) (at 171.7675 67.31 0))
     (property "Value" "LED" (id 1) (at 171.7675 69.85 0))
-    (property "Footprint" "LED_SMD:LED_0603_1608Metric" (id 2) (at 170.18 74.93 0)
+    (property "Footprint" "LED_SMD:LED_0603_1608Metric_Pad1.05x0.95mm_HandSolder" (id 2) (at 170.18 74.93 0)
       (effects (font (size 1.27 1.27)) hide)
     )
@@
     (property "Reference" "R4" (id 0) (at 153.67 82.55 90))
     (property "Value" "2.2k" (id 1) (at 160.02 83.82 90))
-    (property "Footprint" "Resistor_SMD:R_0603_1608Metric" (id 2) (at 153.67 84.328 90)
+    (property "Footprint" "Resistor_SMD:R_0603_1608Metric_Pad0.98x0.95mm_HandSolder" (id 2) (at 153.67 84.328 90)
       (effects (font (size 1.27 1.27)) hide)
     )
@@
       (effects (font (size 1.27 1.27)) (justify left))
     )
-    (property "Footprint" "Capacitor_SMD:C_0201_0603Metric_Pad0.64x0.40mm_HandSolder" (id 2) (at 35.2552 57.15 0)
+    (property "Footprint" "Capacitor_SMD:C_0603_1608Metric_Pad1.08x0.95mm_HandSolder" (id 2) (at 35.2552 57.15 0)
       (effects (font (size 1.27 1.27)) hide)
     )
@@
     (property "Reference" "R5" (id 0) (at 153.67 85.09 90))
     (property "Value" "2.2k" (id 1) (at 160.02 86.36 90))
-    (property "Footprint" "Resistor_SMD:R_0603_1608Metric" (id 2) (at 153.67 86.868 90)
+    (property "Footprint" "Resistor_SMD:R_0603_1608Metric_Pad0.98x0.95mm_HandSolder" (id 2) (at 153.67 86.868 90)
       (effects (font (size 1.27 1.27)) hide)
     )
@@
     (property "Reference" "R2" (id 0) (at 97.79 133.35 90))
     (property "Value" "2.2k" (id 1) (at 101.6 133.35 90))
-    (property "Footprint" "Resistor_SMD:R_0603_1608Metric" (id 2) (at 99.06 137.668 90)
+    (property "Footprint" "Resistor_SMD:R_0603_1608Metric_Pad0.98x0.95mm_HandSolder" (id 2) (at 99.06 137.668 90)
       (effects (font (size 1.27 1.27)) hide)
     )
@@
     (property "Reference" "R37" (id 0) (at 182.88 74.93 90))
     (property "Value" "2.2k" (id 1) (at 189.23 76.2 90))
-    (property "Footprint" "Resistor_SMD:R_0603_1608Metric" (id 2) (at 182.88 76.708 90)
+    (property "Footprint" "Resistor_SMD:R_0603_1608Metric_Pad0.98x0.95mm_HandSolder" (id 2) (at 182.88 76.708 90)
       (effects (font (size 1.27 1.27)) hide)
     )
@@
     (property "Reference" "R36" (id 0) (at 182.88 72.39 90))
     (property "Value" "2.2k" (id 1) (at 189.23 73.66 90))
-    (property "Footprint" "Resistor_SMD:R_0603_1608Metric" (id 2) (at 182.88 74.168 90)
-      (effects (font (size 1.27 1.27)) hide)
-    )
+    (property "Footprint" "Resistor_SMD:R_0603_1608Metric_Pad0.98x0.95mm_HandSolder" (id 2) (at 182.88 74.168 90)
+      (effects (font (size 1.27 1.27)) hide)
+    )

Commit message: full 3d models, pre-routing, corrections
kurwa bezpiecznik od wczoraj a fura dalej nie jeździ siedze u rakietowcow bo cieplo chlopaki co z wami
Connections:
- net CAN-H renamed CAN+
- net CAN+: now also D2.1 (A1); no longer D2.2 (A2)
- net CAN-L renamed CAN-
- net CAN-: now also D2.2 (A2); no longer D2.1 (A1)
Other:
- moved on the sheet: D2
Changed lines of the file:
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@@
     )
   )
-  (global_label "CAN-H" (shape bidirectional) (at 266.7 90.17 0) (fields_autoplaced)
-    (effects (font (size 1.27 1.27)) (justify left))
-    (property "Intersheet References" "${INTERSHEET_REFS}" (id 0) (at 275.705 90.0906 0)
+  (global_label "CAN+" (shape bidirectional) (at 266.7 90.17 0) (fields_autoplaced)
+    (effects (font (size 1.27 1.27)) (justify left))
+    (property "Intersheet References" "${INTERSHEET_REFS}" (id 0) (at 274.3745 90.0906 0)
       (effects (font (size 1.27 1.27)) (justify left) hide)
     )
@@
     )
   )
-  (global_label "CAN-L" (shape bidirectional) (at 266.7 110.49 0) (fields_autoplaced)
-    (effects (font (size 1.27 1.27)) (justify left))
-    (property "Intersheet References" "${INTERSHEET_REFS}" (id 0) (at 275.4026 110.4106 0)
+  (global_label "CAN-" (shape bidirectional) (at 266.7 110.49 0) (fields_autoplaced)
+    (effects (font (size 1.27 1.27)) (justify left))
+    (property "Intersheet References" "${INTERSHEET_REFS}" (id 0) (at 274.3745 110.4106 0)
       (effects (font (size 1.27 1.27)) (justify left) hide)
     )
@@
     (pin "1")
   )
-  (symbol (lib_id "Device:D_TVS_Dual_AAC") (at 255.27 100.33 90) (unit 1)
-    (in_bom yes) (on_board yes)
-    (property "Reference" "D2" (id 0) (at 252.73 99.0599 90)
-      (effects (font (size 1.27 1.27)) (justify left))
-    )
-    (property "Value" "PESD2CAN.215" (id 1) (at 254 101.6 90)
-      (effects (font (size 1.27 1.27)) (justify left))
-    )
-    (property "Footprint" "Package_TO_SOT_SMD:SOT-23" (id 2) (at 255.27 104.14 0)
-      (effects (font (size 1.27 1.27)) hide)
-    )
-    (property "Datasheet" "~" (id 3) (at 255.27 104.14 0)
+  (symbol (lib_id "Device:D_TVS_Dual_AAC") (at 255.27 100.33 270) (unit 1)
+    (in_bom yes) (on_board yes)
+    (property "Reference" "D2" (id 0) (at 257.81 101.6001 90)
+      (effects (font (size 1.27 1.27)) (justify left))
+    )
+    (property "Value" "PESD2CAN.215" (id 1) (at 247.65 113.03 90)
+      (effects (font (size 1.27 1.27)) (justify left))
+    )
+    (property "Footprint" "Package_TO_SOT_SMD:SOT-23" (id 2) (at 255.27 96.52 0)
+      (effects (font (size 1.27 1.27)) hide)
+    )
+    (property "Datasheet" "~" (id 3) (at 255.27 96.52 0)
       (effects (font (size 1.27 1.27)) hide)
     )
@@
     (pin "2")
   )
-  (symbol (lib_id "power:GND") (at 259.08 100.33 0) (unit 1)
-    (in_bom yes) (on_board yes)
-    (property "Reference" "#PWR029" (id 0) (at 259.08 106.68 0)
-      (effects (font (size 1.27 1.27)) hide)
-    )
-    (property "Value" "GND" (id 1) (at 259.207 104.7242 0))
-    (property "Footprint" "" (id 2) (at 259.08 100.33 0)
-      (effects (font (size 1.27 1.27)) hide)
-    )
-    (property "Datasheet" "" (id 3) (at 259.08 100.33 0)
-      (effects (font (size 1.27 1.27)) hide)
-    )
+  (symbol (lib_id "power:GND") (at 251.46 100.33 270) (unit 1)
+    (in_bom yes) (on_board yes)
+    (property "Reference" "#PWR029" (id 0) (at 245.11 100.33 0)
+      (effects (font (size 1.27 1.27)) hide)
+    )
+    (property "Value" "GND" (id 1) (at 247.0658 100.457 0))
+    (property "Footprint" "" (id 2) (at 251.46 100.33 0)
+      (effects (font (size 1.27 1.27)) hide)
+    )
+    (property "Datasheet" "" (id 3) (at 251.46 100.33 0)
+      (effects (font (size 1.27 1.27)) hide)
+    )

Commit message: still working
Parts:
- added D6: LED, LED_SMD:LED_0603_1608Metric_Pad1.05x0.95mm_HandSolder, symbol Device:LED
- added R47: 2.2k, Resistor_SMD:R_0603_1608Metric_Pad0.98x0.95mm_HandSolder, symbol Device:R
Connections:
- net CAN+: now also D2.2 (A2); no longer D2.1 (A1)
- net CAN-: now also D2.1 (A1); no longer D2.2 (A2)
- net CHECKUP: now reaches U5.17 (PA3)
- net CHECKUP: now also D6.2 (A)
- new net: D6.1 (K), R47.1
- no-connect marks 31 -> 30
Other:
- moved on the sheet: D16, D17, D18, D2
Changed lines of the file:
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@@
   (junction (at 129.54 59.182) (diameter 0) (color 0 0 0 0)
   )
-  (no_connect (at 144.78 77.47))
   (no_connect (at 144.78 151.13))
   (no_connect (at 144.78 130.81))
@@
     (stroke (width 0) (type default) (color 0 0 0 0))
   )
-  (wire (pts (xy 144.78 69.85) (xy 153.67 69.85))
+  (wire (pts (xy 144.78 69.85) (xy 152.4 69.85))
     (stroke (width 0) (type default) (color 0 0 0 0))
   )
@@
     (stroke (width 0) (type default) (color 0 0 0 0))
   )
+  (wire (pts (xy 176.53 77.47) (xy 179.07 77.47))
+    (stroke (width 0) (type default) (color 0 0 0 0))
+  )
   (wire (pts (xy 34.29 57.15) (xy 34.29 63.5))
     (stroke (width 0) (type default) (color 0 0 0 0))
@@
     (stroke (width 0) (type default) (color 0 0 0 0))
   )
-  (wire (pts (xy 161.29 69.85) (xy 179.07 69.85))
+  (wire (pts (xy 160.02 69.85) (xy 179.07 69.85))
     (stroke (width 0) (type default) (color 0 0 0 0))
   )
@@
     (stroke (width 0) (type default) (color 0 0 0 0))
   )
+  (wire (pts (xy 144.78 77.47) (xy 168.91 77.47))
+    (stroke (width 0) (type default) (color 0 0 0 0))
+  )
   (polyline (pts (xy 187.96 88.9) (xy 210.82 88.9))
     (stroke (width 0) (type default) (color 0 0 0 0))
@@
     (stroke (width 0) (type default) (color 0 0 0 0))
   )
+  (wire (pts (xy 186.69 77.47) (xy 198.12 77.47))
+    (stroke (width 0) (type default) (color 0 0 0 0))
+  )
   (wire (pts (xy 262.89 90.17) (xy 266.7 90.17))
     (stroke (width 0) (type default) (color 0 0 0 0))
@@
     (stroke (width 0) (type default) (color 0 0 0 0))
   )
-  (wire (pts (xy 167.64 72.39) (xy 179.07 72.39))
+  (wire (pts (xy 165.1 72.39) (xy 179.07 72.39))
     (stroke (width 0) (type default) (color 0 0 0 0))
   )
@@
     (stroke (width 0) (type default) (color 0 0 0 0))
   )
-  (wire (pts (xy 144.78 74.93) (xy 166.37 74.93))
+  (wire (pts (xy 144.78 74.93) (xy 162.56 74.93))
     (stroke (width 0) (type default) (color 0 0 0 0))
   )
@@
     (stroke (width 0) (type default) (color 0 0 0 0))
   )
-  (wire (pts (xy 173.99 74.93) (xy 179.07 74.93))
+  (wire (pts (xy 170.18 74.93) (xy 179.07 74.93))
     (stroke (width 0) (type default) (color 0 0 0 0))
   )
@@
     (stroke (width 0) (type default) (color 0 0 0 0))
   )
-  (wire (pts (xy 144.78 72.39) (xy 160.02 72.39))
+  (wire (pts (xy 144.78 72.39) (xy 157.48 72.39))
     (stroke (width 0) (type default) (color 0 0 0 0))
   )
@@
   )
   (label "ERROR" (at 149.86 74.93 0)
+    (effects (font (size 1.27 1.27)) (justify left bottom))
+  )
+  (label "CHECKUP" (at 149.86 77.47 0)
     (effects (font (size 1.27 1.27)) (justify left bottom))
   )
@@
     (pin "1")
   )
-  (symbol (lib_id "Device:D_TVS_Dual_AAC") (at 255.27 100.33 270) (unit 1)
-    (in_bom yes) (on_board yes)
-    (property "Reference" "D2" (id 0) (at 257.81 101.6001 90)
-      (effects (font (size 1.27 1.27)) (justify left))
-    )
-    (property "Value" "PESD2CAN.215" (id 1) (at 247.65 113.03 90)
-      (effects (font (size 1.27 1.27)) (justify left))
-    )
-    (property "Footprint" "Package_TO_SOT_SMD:SOT-23" (id 2) (at 255.27 96.52 0)
-      (effects (font (size 1.27 1.27)) hide)
-    )
-    (property "Datasheet" "~" (id 3) (at 255.27 96.52 0)
+  (symbol (lib_id "Device:D_TVS_Dual_AAC") (at 255.27 100.33 90) (unit 1)
+    (in_bom yes) (on_board yes)
+    (property "Reference" "D2" (id 0) (at 252.73 99.0599 90)
+      (effects (font (size 1.27 1.27)) (justify left))
+    )
+    (property "Value" "PESD2CAN.215" (id 1) (at 262.89 87.63 90)
+      (effects (font (size 1.27 1.27)) (justify left))
+    )
+    (property "Footprint" "Package_TO_SOT_SMD:SOT-23" (id 2) (at 255.27 104.14 0)
+      (effects (font (size 1.27 1.27)) hide)
+    )
+    (property "Datasheet" "~" (id 3) (at 255.27 104.14 0)
       (effects (font (size 1.27 1.27)) hide)
     )
@@
     (pin "3")
   )
-  (symbol (lib_id "Device:LED") (at 157.48 69.85 180) (unit 1)
+  (symbol (lib_id "Device:LED") (at 156.21 69.85 180) (unit 1)
     (in_bom yes) (on_board yes) (fields_autoplaced)
-    (property "Reference" "D16" (id 0) (at 159.0675 62.23 0))
-    (property "Value" "LED" (id 1) (at 159.0675 64.77 0))
-    (property "Footprint" "LED_SMD:LED_0603_1608Metric_Pad1.05x0.95mm_HandSolder" (id 2) (at 157.48 69.85 0)
-      (effects (font (size 1.27 1.27)) hide)
-    )
-    (property "Datasheet" "~" (id 3) (at 157.48 69.85 0)
+    (property "Reference" "D16" (id 0) (at 157.7975 62.23 0))
+    (property "Value" "LED" (id 1) (at 157.7975 64.77 0))
+    (property "Footprint" "LED_SMD:LED_0603_1608Metric_Pad1.05x0.95mm_HandSolder" (id 2) (at 156.21 69.85 0)
+      (effects (font (size 1.27 1.27)) hide)
+    )
+    (property "Datasheet" "~" (id 3) (at 156.21 69.85 0)
       (effects (font (size 1.27 1.27)) hide)
     )
@@
     (pin "1")
   )
-  (symbol (lib_id "Device:LED") (at 163.83 72.39 180) (unit 1)
-    (in_bom yes) (on_board yes) (fields_autoplaced)
-    (property "Reference" "D17" (id 0) (at 165.4175 64.77 0))
-    (property "Value" "LED" (id 1) (at 165.4175 67.31 0))
-    (property "Footprint" "LED_SMD:LED_0603_1608Metric_Pad1.05x0.95mm_HandSolder" (id 2) (at 163.83 72.39 0)
-      (effects (font (size 1.27 1.27)) hide)
-    )
-    (property "Datasheet" "~" (id 3) (at 163.83 72.39 0)
+  (symbol (lib_id "Device:LED") (at 161.29 72.39 180) (unit 1)
+    (in_bom yes) (on_board yes)
+    (property "Reference" "D17" (id 0) (at 163.83 64.77 0))
+    (property "Value" "LED" (id 1) (at 163.83 67.31 0))
+    (property "Footprint" "LED_SMD:LED_0603_1608Metric_Pad1.05x0.95mm_HandSolder" (id 2) (at 161.29 72.39 0)
+      (effects (font (size 1.27 1.27)) hide)
+    )
+    (property "Datasheet" "~" (id 3) (at 161.29 72.39 0)
       (effects (font (size 1.27 1.27)) hide)
     )
@@
     (pin "2")
   )
-  (symbol (lib_id "Device:LED") (at 170.18 74.93 180) (unit 1)
-    (in_bom yes) (on_board yes) (fields_autoplaced)
-    (property "Reference" "D18" (id 0) (at 171.7675 67.31 0))
-    (property "Value" "LED" (id 1) (at 171.7675 69.85 0))
-    (property "Footprint" "LED_SMD:LED_0603_1608Metric_Pad1.05x0.95mm_HandSolder" (id 2) (at 170.18 74.93 0)
-      (effects (font (size 1.27 1.27)) hide)
-    )
-    (property "Datasheet" "~" (id 3) (at 170.18 74.93 0)
+  (symbol (lib_id "Device:LED") (at 166.37 74.93 180) (unit 1)
+    (in_bom yes) (on_board yes)
+    (property "Reference" "D18" (id 0) (at 168.91 68.58 0))
+    (property "Value" "LED" (id 1) (at 168.91 71.12 0))
+    (property "Footprint" "LED_SMD:LED_0603_1608Metric_Pad1.05x0.95mm_HandSolder" (id 2) (at 166.37 74.93 0)
+      (effects (font (size 1.27 1.27)) hide)
+    )
+    (property "Datasheet" "~" (id 3) (at 166.37 74.93 0)
       (effects (font (size 1.27 1.27)) hide)
     )
@@
     (pin "2")
   )
-  (symbol (lib_id "power:GND") (at 251.46 100.33 270) (unit 1)
-    (in_bom yes) (on_board yes)
-    (property "Reference" "#PWR029" (id 0) (at 245.11 100.33 0)
-      (effects (font (size 1.27 1.27)) hide)
-    )
-    (property "Value" "GND" (id 1) (at 247.0658 100.457 0))
-    (property "Footprint" "" (id 2) (at 251.46 100.33 0)
-      (effects (font (size 1.27 1.27)) hide)
-    )
-    (property "Datasheet" "" (id 3) (at 251.46 100.33 0)
+  (symbol (lib_id "Device:R") (at 182.88 77.47 90) (unit 1)
+    (in_bom yes) (on_board yes)
+    (property "Reference" "R47" (id 0) (at 182.88 77.47 90))
+    (property "Value" "2.2k" (id 1) (at 189.23 78.74 90))
+    (property "Footprint" "Resistor_SMD:R_0603_1608Metric_Pad0.98x0.95mm_HandSolder" (id 2) (at 182.88 79.248 90)
+      (effects (font (size 1.27 1.27)) hide)
+    )
+    (property "Datasheet" "~" (id 3) (at 182.88 77.47 0)
+      (effects (font (size 1.27 1.27)) hide)
+    )
+    (pin "1")
+    (pin "2")
+  )
+  (symbol (lib_id "power:GND") (at 259.08 100.33 0) (unit 1)
+    (in_bom yes) (on_board yes)
+    (property "Reference" "#PWR029" (id 0) (at 259.08 106.68 0)
+      (effects (font (size 1.27 1.27)) hide)
+    )
+    (property "Value" "GND" (id 1) (at 259.207 104.7242 0))
+    (property "Footprint" "" (id 2) (at 259.08 100.33 0)
+      (effects (font (size 1.27 1.27)) hide)
+    )
+    (property "Datasheet" "" (id 3) (at 259.08 100.33 0)
       (effects (font (size 1.27 1.27)) hide)
     )
@@
       (effects (font (size 1.27 1.27)) hide)
     )
+    (pin "1")
+    (pin "2")
+  )
+  (symbol (lib_id "Device:LED") (at 172.72 77.47 180) (unit 1)
+    (in_bom yes) (on_board yes)
+    (property "Reference" "D6" (id 0) (at 175.26 71.12 0))
+    (property "Value" "LED" (id 1) (at 175.26 73.66 0))
+    (property "Footprint" "LED_SMD:LED_0603_1608Metric_Pad1.05x0.95mm_HandSolder" (id 2) (at 172.72 77.47 0)
+      (effects (font (size 1.27 1.27)) hide)
+    )
+    (property "Datasheet" "~" (id 3) (at 172.72 77.47 0)
+      (effects (font (size 1.27 1.27)) hide)
+    )

Commit message: kurde no jeszcze nie skonczylem ale sune dalej
Connections:
- net CAN_RX renamed CAN_RX+
- net CAN_TX renamed CAN_TX-
Changed lines of the file:
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@@
     (effects (font (size 1.27 1.27)) (justify left bottom))
   )
-  (label "CAN_TX" (at 199.39 95.25 0)
+  (label "CAN_TX-" (at 199.39 95.25 0)
     (effects (font (size 1.27 1.27)) (justify left bottom))
   )
-  (label "CAN_TX" (at 158.75 100.33 180)
+  (label "CAN_TX-" (at 158.75 100.33 180)
     (effects (font (size 1.27 1.27)) (justify right bottom))
   )
@@
     (effects (font (size 1.27 1.27)) (justify left bottom))
   )
-  (label "CAN_RX" (at 158.75 97.79 180)
+  (label "CAN_RX+" (at 158.75 97.79 180)
     (effects (font (size 1.27 1.27)) (justify right bottom))
   )
@@
     (effects (font (size 1.27 1.27)) (justify right bottom))
   )
-  (label "CAN_RX" (at 199.39 97.79 0)
+  (label "CAN_RX+" (at 199.39 97.79 0)
     (effects (font (size 1.27 1.27)) (justify left bottom))
   )

Commit message: wip
Connections:
- net GND: now also R47.2
Changed lines of the file:
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@@
   (junction (at 127 159.258) (diameter 0) (color 0 0 0 0)
+  )
+  (junction (at 198.12 77.47) (diameter 0) (color 0 0 0 0)
   )
   (junction (at 227.33 78.74) (diameter 0) (color 0 0 0 0)
@@
     (stroke (width 0) (type default) (color 0 0 0 0))
   )
+  (wire (pts (xy 198.12 77.47) (xy 198.12 78.74))
+    (stroke (width 0) (type default) (color 0 0 0 0))
+  )
   (wire (pts (xy 255.27 110.49) (xy 262.89 110.49))
     (stroke (width 0) (type default) (color 0 0 0 0))
@@
     (stroke (width 0) (type default) (color 0 0 0 0))
   )
-  (wire (pts (xy 198.12 74.93) (xy 198.12 76.2))
+  (wire (pts (xy 198.12 74.93) (xy 198.12 77.47))
     (stroke (width 0) (type default) (color 0 0 0 0))
   )
@@
     (effects (font (size 1.27 1.27)) (justify right bottom))
   )
-  (label "ERROR" (at 149.86 74.93 0)
-    (effects (font (size 1.27 1.27)) (justify left bottom))
-  )
-  (label "CHECKUP" (at 149.86 77.47 0)
+  (label "ERROR" (at 148.59 74.93 0)
+    (effects (font (size 1.27 1.27)) (justify left bottom))
+  )
+  (label "CHECKUP" (at 148.59 77.47 0)
     (effects (font (size 1.27 1.27)) (justify left bottom))
   )
@@
     (pin "1")
   )
-  (symbol (lib_id "power:GND") (at 198.12 76.2 0) (unit 1)
+  (symbol (lib_id "power:GND") (at 198.12 78.74 0) (unit 1)
     (in_bom yes) (on_board yes) (fields_autoplaced)
-    (property "Reference" "#PWR02" (id 0) (at 198.12 82.55 0)
-      (effects (font (size 1.27 1.27)) hide)
-    )
-    (property "Value" "GND" (id 1) (at 198.12 81.28 0))
-    (property "Footprint" "" (id 2) (at 198.12 76.2 0)
-      (effects (font (size 1.27 1.27)) hide)
-    )
-    (property "Datasheet" "" (id 3) (at 198.12 76.2 0)
-      (effects (font (size 1.27 1.27)) hide)
-    )
+    (property "Reference" "#PWR02" (id 0) (at 198.12 85.09 0)
+      (effects (font (size 1.27 1.27)) hide)
+    )
+    (property "Value" "GND" (id 1) (at 198.12 83.82 0))
+    (property "Footprint" "" (id 2) (at 198.12 78.74 0)
+      (effects (font (size 1.27 1.27)) hide)
+    )
+    (property "Datasheet" "" (id 3) (at 198.12 78.74 0)
+      (effects (font (size 1.27 1.27)) hide)
+    )

Commit message: fixed references addet tp;s mam pojutrze przejebany egzamin nara
Parts:
- added NT1: NetTie_2, NetTie:NetTie-2_SMD_Pad0.5mm, symbol Device:NetTie_2
Connections:
- net +3V3: now also NT1.1
- net 3V3_SYS: now also NT1.2
- net AIR_MAIN: now also U5.8 (PC0); no longer U5.10 (PC2)
- net AIR_REDUNDANT: now also U5.10 (PC2); no longer U5.8 (PC0)
- net AS_CLOSE_SDC: now also R4.2; no longer R5.2
- net WATCHDOG: now also R5.2; no longer R4.2
- net CAN_RX+ renamed (CAN_RX)+
- net CAN_TX- renamed (CAN_TX)-

Commit message: supply section redesign due to IC shortage
Parts:
- Y1: footprint Crystal:Crystal_SMD_2520-4Pin_2.5x2.0mm -> Crystal:Crystal_SMD_3225-4Pin_3.2x2.5mm
Changed lines of the file:
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@@
     (property "Reference" "Y1" (id 0) (at 46.228 98.298 0))
     (property "Value" "Crystal_GND24" (id 1) (at 51.562 100.584 0))
-    (property "Footprint" "Crystal:Crystal_SMD_2520-4Pin_2.5x2.0mm" (id 2) (at 64.77 102.87 0)
+    (property "Footprint" "Crystal:Crystal_SMD_3225-4Pin_3.2x2.5mm" (id 2) (at 64.77 102.87 0)
       (effects (font (size 1.27 1.27)) hide)
     )
