File: hardware/buffer.kicad_sch (KiCad schematic)
At the start: 7 parts, among them U8 OPA365xxD

Commit message: WIP revision 2 layout refinement
Parts:
- removed U8: OPA365xxD, Package_SO:SOIC-8_3.9x4.9mm_P1.27mm, symbol Amplifier_Operational:OPA365xxD
- added U1: OPA365xxDBV, Package_TO_SOT_SMD:SOT-23-5, symbol Amplifier_Operational:OPA365xxDBV
Connections:
- net +3V3: now also U1.5 (V+)
- net GND: now also U1.2 (V-)
- net opa_output: now also U1.1
- net at R24.2, R38.1: now also U1.3 (+)
- net at C25.1, R21.2, R41.1: now also U1.4 (-)
Changed lines of the file:
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@@
-    )
-  )
-  (symbol (lib_id "Amplifier_Operational:OPA365xxD") (at 152.4 88.9 0) (unit 1)
-    (in_bom yes) (on_board yes) (dnp no)
-    (property "Reference" "U8" (at 156.21 82.55 0)
-      (effects (font (size 1.27 1.27)))
-    )
-    (property "Value" "OPA365xxD" (at 157.48 85.09 0)
-      (effects (font (size 1.27 1.27)))
-    )
-    (property "Footprint" "Package_SO:SOIC-8_3.9x4.9mm_P1.27mm" (at 149.86 93.98 0)
-      (effects (font (size 1.27 1.27)) (justify left) hide)
-    )
-    (property "Datasheet" "http://www.ti.com/lit/ds/symlink/opa365.pdf" (at 156.21 85.09 0)
-      (effects (font (size 1.27 1.27)) hide)
-    )
-    (pin "1")
-    (pin "2")
-    (pin "3")
-    (pin "4")
-    (pin "5")
-    (pin "6")
-    (pin "7")
-    (pin "8")
-    (instances
-      (project "PUTM_DV_EBS_2023"
-        (path "/d921fbb5-521e-405d-bdec-f40195adfa1c/0e6e746e-cf7c-47e8-8ed6-c681697efa7a/ae830780-2461-4e8c-b528-b01e34f9f141"
-          (reference "U8") (unit 1)
-        )
-        (path "/d921fbb5-521e-405d-bdec-f40195adfa1c/0e6e746e-cf7c-47e8-8ed6-c681697efa7a/2138a410-a835-4c5b-94a4-707f9fcacbbd"
-          (reference "U9") (unit 1)
-        )
-        (path "/d921fbb5-521e-405d-bdec-f40195adfa1c/0e6e746e-cf7c-47e8-8ed6-c681697efa7a/d2cebea6-4b71-4d4d-8083-65636bff8f5a"
-          (reference "U10") (unit 1)
-        )
-        (path "/d921fbb5-521e-405d-bdec-f40195adfa1c/0e6e746e-cf7c-47e8-8ed6-c681697efa7a/f266ff56-9481-481d-8224-0f0c95f197a3"
-          (reference "U12") (unit 1)
-        )
-      )
     )
   )
@@
         )
       )
+    )
+  )
+  (symbol (lib_id "Amplifier_Operational:OPA365xxDBV") (at 152.4 88.9 0) (unit 1)
+    (in_bom yes) (on_board yes) (dnp no) (fields_autoplaced)
+    (property "Reference" "U1" (at 165.1 85.4711 0)
+      (effects (font (size 1.27 1.27)))
+    )
+    (property "Value" "OPA365xxDBV" (at 165.1 88.0111 0)
+      (effects (font (size 1.27 1.27)))
+    )
+    (property "Footprint" "Package_TO_SOT_SMD:SOT-23-5" (at 149.86 93.98 0)
+      (effects (font (size 1.27 1.27)) (justify left) hide)
+    )
+    (property "Datasheet" "https://www.ti.com/lit/ds/symlink/opa365.pdf" (at 152.4 83.82 0)
+      (effects (font (size 1.27 1.27)) hide)
+    )
+    (pin "2")
+    (pin "5")
+    (pin "1")
+    (pin "3")
+    (pin "4")
+    (instances
+      (project "PUTM_DV_EBS_2023"
+        (path "/d921fbb5-521e-405d-bdec-f40195adfa1c/0e6e746e-cf7c-47e8-8ed6-c681697efa7a/ae830780-2461-4e8c-b528-b01e34f9f141"
+          (reference "U1") (unit 1)
+        )
+        (path "/d921fbb5-521e-405d-bdec-f40195adfa1c/0e6e746e-cf7c-47e8-8ed6-c681697efa7a/2138a410-a835-4c5b-94a4-707f9fcacbbd"
+          (reference "U2") (unit 1)
+        )
+        (path "/d921fbb5-521e-405d-bdec-f40195adfa1c/0e6e746e-cf7c-47e8-8ed6-c681697efa7a/d2cebea6-4b71-4d4d-8083-65636bff8f5a"
+          (reference "U3") (unit 1)
+        )
+        (path "/d921fbb5-521e-405d-bdec-f40195adfa1c/0e6e746e-cf7c-47e8-8ed6-c681697efa7a/f266ff56-9481-481d-8224-0f0c95f197a3"
+          (reference "U4") (unit 1)
+        )
+      )

Commit message: Dimensions compress, routing
Parts:
- R21, R24: value 200k 1% -> 20k 1%
- R38, R41: value 100k 1% -> 10k 1%
Other:
- note added: "zmniejszyc wartosci rezystorow wykres sprawdzania SCS"
