File: hardware/buffer.kicad_sch (KiCad schematic)
At the start: 7 parts, among them U1 OPA365xxDBV

Commit message: changed pcb version
Parts:
- removed C21: 100n, Capacitor_SMD:C_0603_1608Metric_Pad1.08x0.95mm_HandSolder, symbol Device:C_Small
- removed C25: 10n, Capacitor_SMD:C_0603_1608Metric_Pad1.08x0.95mm_HandSolder, symbol Device:C
- removed R21, R24: 20k 1%, Resistor_SMD:R_0603_1608Metric_Pad0.98x0.95mm_HandSolder, symbol Device:R
- removed R41: 10k 1%, Resistor_SMD:R_0603_1608Metric_Pad0.98x0.95mm_HandSolder, symbol Device:R
- removed U1: OPA365xxDBV, Package_TO_SOT_SMD:SOT-23-5, symbol Amplifier_Operational:OPA365xxDBV
- added C34: 5.6n, Capacitor_SMD:C_0603_1608Metric_Pad1.08x0.95mm_HandSolder, symbol Device:C
- added C37: 100nF, Capacitor_SMD:C_0603_1608Metric, symbol Device:C
- added R39: 6.8k 1%, Resistor_SMD:R_0603_1608Metric_Pad0.98x0.95mm_HandSolder, symbol Device:R
- added R40: 1k, Resistor_SMD:R_0603_1608Metric_Pad0.98x0.95mm_HandSolder, symbol Device:R
- added U8: TSX7191, Package_TO_SOT_SMD:SOT-23-5_HandSoldering, symbol Simulation_SPICE:OPAMP
- R38: value 10k 1% -> 3.3k 1%
Connections:
- net GND: now also C34.2, C37.2, R39.2, U8.5 (V-); no longer R38.2
- net AIR_R: now reaches R38.1
- new net: C34.1, R38.2, R39.1, U8.1 (+)
- new net: R40.1, U8.2 (-), U8.3
- new net +5V: C37.1, U8.4 (V+)
- new net AIR_SENSOR: R40.2
Other:
- note added: "1k(sens out z)"
- note added: "PSE output impedance= 1kOhm"
- note removed: "//5V input to 2.5V output analog level shifter"
- note removed: "zmniejszyc wartosci rezystorow wykres sprawdzania SCS"

Commit message: uploaded older pcb version
Parts:
- U8: value TSX7191 -> ${SIM.PARAMS}; Spice_Netlist_Enabled Y -> (none); Spice_Primitive X -> (none)
