File: hardware/decoupling.kicad_sch (KiCad schematic)
At the start: 8 parts

Commit message: replace RES2 input to actuator relai
Parts:
- removed C8: 100nF, Capacitor_SMD:C_0603_1608Metric_Pad1.08x0.95mm_HandSolder, symbol Device:C
Other:
- moved on the sheet: L1
Changed lines of the file:
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@@
   (junction (at 138.43 90.17) (diameter 0) (color 0 0 0 0)
   )
+  (junction (at 115.57 90.17) (diameter 0) (color 0 0 0 0)
+  )
   (junction (at 149.86 90.17) (diameter 0) (color 0 0 0 0)
   )
-  (junction (at 127 90.17) (diameter 0) (color 0 0 0 0)
-  )
-  (junction (at 119.38 90.17) (diameter 0) (color 0 0 0 0)
-  )
   (junction (at 161.29 90.17) (diameter 0) (color 0 0 0 0)
   )
@@
     (stroke (width 0) (type default))
   )
-  (wire (pts (xy 127 99.06) (xy 127 105.41))
+  (wire (pts (xy 115.57 90.17) (xy 125.73 90.17))
     (stroke (width 0) (type default))
   )
@@
     (stroke (width 0) (type default))
   )
-  (wire (pts (xy 119.38 80.01) (xy 119.38 90.17))
+  (wire (pts (xy 115.57 80.01) (xy 115.57 90.17))
     (stroke (width 0) (type default))
   )
@@
     (stroke (width 0) (type default))
   )
-  (wire (pts (xy 138.43 90.17) (xy 127 90.17))
+  (wire (pts (xy 138.43 90.17) (xy 133.35 90.17))
     (stroke (width 0) (type default))
   )
@@
     (stroke (width 0) (type default))
   )
-  (wire (pts (xy 115.57 90.17) (xy 119.38 90.17))
-    (stroke (width 0) (type default))
-  )
   (wire (pts (xy 173.99 90.17) (xy 173.99 91.44))
     (stroke (width 0) (type default))
   )
-  (wire (pts (xy 127 90.17) (xy 127 91.44))
-    (stroke (width 0) (type default))
-  )
-  (label "3v3_A" (at 119.38 80.01 90) (fields_autoplaced)
-    (effects (font (size 1.27 1.27)) (justify left bottom))
-  )
-  (symbol (lib_id "power:GND") (at 127 105.41 0) (unit 1)
-    (in_bom yes) (on_board yes) (dnp no)
-    (property "Reference" "#PWR018" (at 127 111.76 0)
-      (effects (font (size 1.27 1.27)) hide)
-    )
-    (property "Value" "GND" (at 127 110.49 0)
-      (effects (font (size 1.27 1.27)))
-    )
-    (property "Footprint" "" (at 127 105.41 0)
-      (effects (font (size 1.27 1.27)) hide)
-    )
-    (property "Datasheet" "" (at 127 105.41 0)
-      (effects (font (size 1.27 1.27)) hide)
-    )
-    (pin "1")
-    (instances
-      (project "PUTM_DV_EBS_2023"
-        (path "/d921fbb5-521e-405d-bdec-f40195adfa1c/bbd4f989-bc6f-4d23-b657-5429a2409e1d"
-          (reference "#PWR018") (unit 1)
-        )
-        (path "/d921fbb5-521e-405d-bdec-f40195adfa1c/bbd4f989-bc6f-4d23-b657-5429a2409e1d/cb98bda1-8cc2-4b83-bddd-d5756e33cfe1"
-          (reference "#PWR017") (unit 1)
-        )
-      )
+  (global_label "3v3_A" (shape input) (at 115.57 80.01 90) (fields_autoplaced)
+    (effects (font (size 1.27 1.27)) (justify left))
+    (property "Intersheetrefs" "${INTERSHEET_REFS}" (at 115.57 71.6614 90)
+      (effects (font (size 1.27 1.27)) (justify left) hide)
     )
   )
@@
     )
   )
-  (symbol (lib_id "Device:L") (at 123.19 90.17 90) (unit 1)
-    (in_bom yes) (on_board yes) (dnp no)
-    (property "Reference" "L1" (at 122.0216 88.8238 0)
-      (effects (font (size 1.27 1.27)) (justify left))
-    )
-    (property "Value" "10u" (at 124.333 88.8238 0)
-      (effects (font (size 1.27 1.27)) (justify left))
-    )
-    (property "Footprint" "Inductor_SMD:L_0805_2012Metric" (at 123.19 90.17 0)
-      (effects (font (size 1.27 1.27)) hide)
-    )
-    (property "Datasheet" "~" (at 123.19 90.17 0)
+  (symbol (lib_id "Device:L") (at 129.54 90.17 90) (unit 1)
+    (in_bom yes) (on_board yes) (dnp no)
+    (property "Reference" "L1" (at 128.3716 88.8238 0)
+      (effects (font (size 1.27 1.27)) (justify left))
+    )
+    (property "Value" "10u" (at 130.683 88.8238 0)
+      (effects (font (size 1.27 1.27)) (justify left))
+    )
+    (property "Footprint" "Inductor_SMD:L_0805_2012Metric" (at 129.54 90.17 0)
+      (effects (font (size 1.27 1.27)) hide)
+    )
+    (property "Datasheet" "~" (at 129.54 90.17 0)
       (effects (font (size 1.27 1.27)) hide)
     )
@@
         )
       )
-    )
-  )
-  (symbol (lib_id "Device:C") (at 127 95.25 0) (unit 1)
-    (in_bom yes) (on_board yes) (dnp no)
-    (property "Reference" "C8" (at 129.921 94.0816 0)
-      (effects (font (size 1.27 1.27)) (justify left))
-    )
-    (property "Value" "100nF" (at 129.921 96.393 0)
-      (effects (font (size 1.27 1.27)) (justify left))
-    )
-    (property "Footprint" "Capacitor_SMD:C_0603_1608Metric_Pad1.08x0.95mm_HandSolder" (at 127.9652 99.06 0)
-      (effects (font (size 1.27 1.27)) hide)
-    )
-    (property "Datasheet" "~" (at 127 95.25 0)
-      (effects (font (size 1.27 1.27)) hide)
-    )
-    (pin "1")
-    (pin "2")
-    (instances
-      (project "PUTM_DV_EBS_2023"
-        (path "/d921fbb5-521e-405d-bdec-f40195adfa1c/bbd4f989-bc6f-4d23-b657-5429a2409e1d"
-          (reference "C8") (unit 1)
-        )
-        (path "/d921fbb5-521e-405d-bdec-f40195adfa1c/bbd4f989-bc6f-4d23-b657-5429a2409e1d/cb98bda1-8cc2-4b83-bddd-d5756e33cfe1"
-          (reference "C7") (unit 1)
-        )
-      )
