File: hardware/latch.kicad_sch (KiCad schematic)
At the start: 5 parts, among them K2 FINDER-30.22, Q4 BSS123

Commit message: WIP revision 2 layout refinement
Parts:
- D12: symbol Diode:1N5408 -> Diode:1N5817
Changed lines of the file:
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@@
     (effects (font (size 1.27 1.27)) (justify right))
   )
-  (symbol (lib_id "Diode:1N5408") (at 127 85.09 90) (mirror x) (unit 1)
+  (symbol (lib_id "Diode:1N5817") (at 127 85.09 90) (mirror x) (unit 1)
     (in_bom yes) (on_board yes) (dnp no) (fields_autoplaced)
     (property "Reference" "D12" (at 129.54 83.8199 90)

Commit message: WIP 1.1 routing
Parts:
- R1: value 1k -> 100R
Changed lines of the file:
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@@
       (effects (font (size 1.27 1.27)))
     )
-    (property "Value" "1k" (at 111.76 104.14 90)
+    (property "Value" "100R" (at 111.76 104.14 90)
       (effects (font (size 1.27 1.27)))
     )

Commit message: 2.0 layot wip , routing 3
Parts:
- D12: footprint Diode_SMD:D_SMA_Handsoldering -> Diode_SMD:D_SMA
Changed lines of the file:
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@@
       (effects (font (size 1.27 1.27)) (justify right))
     )
-    (property "Footprint" "Diode_SMD:D_SMA_Handsoldering" (at 131.445 85.09 0)
+    (property "Footprint" "Diode_SMD:D_SMA" (at 131.445 85.09 0)
       (effects (font (size 1.27 1.27)) hide)
     )

Commit message: replace RES2 input to actuator relai
Connections:
- net LINE: no longer names the net of K2.24
- net VALVE_SUPPLY: no longer names the net of K2.21
- no-connect marks 2 -> 4
Other:
- note removed: "LINE means supply connected After LVMS-> ASMS-> RES-> 2 Required by T15 2.2"
Changed lines of the file:
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@@
   (junction (at 143.51 125.73) (diameter 0) (color 0 0 0 0)
-  )
-  (junction (at 166.37 48.26) (diameter 0) (color 0 0 0 0)
   )
   (junction (at 143.51 76.2) (diameter 0) (color 0 0 0 0)
@@
   (junction (at 143.51 95.25) (diameter 0) (color 0 0 0 0)
   )
+  (no_connect (at 163.83 92.71))
   (no_connect (at 161.29 77.47))
   (no_connect (at 151.13 77.47))
+  (no_connect (at 166.37 77.47))
   (wire (pts (xy 143.51 125.73) (xy 143.51 134.62))
     (stroke (width 0) (type default))
   )
   (wire (pts (xy 153.67 104.14) (xy 153.67 92.71))
-    (stroke (width 0) (type default))
-  )
-  (wire (pts (xy 156.21 48.26) (xy 156.21 45.72))
     (stroke (width 0) (type default))
   )
@@
     (stroke (width 0) (type default))
   )
-  (wire (pts (xy 166.37 48.26) (xy 156.21 48.26))
-    (stroke (width 0) (type default))
-  )
   (wire (pts (xy 127 81.28) (xy 127 76.2))
     (stroke (width 0) (type default))
@@
     (stroke (width 0) (type default))
   )
-  (wire (pts (xy 166.37 48.26) (xy 166.37 77.47))
-    (stroke (width 0) (type default))
-  )
-  (wire (pts (xy 163.83 97.79) (xy 163.83 92.71))
-    (stroke (width 0) (type default))
-  )
   (wire (pts (xy 96.52 107.95) (xy 107.95 107.95))
-    (stroke (width 0) (type default))
-  )
-  (wire (pts (xy 201.93 97.79) (xy 163.83 97.79))
     (stroke (width 0) (type default))
   )
@@
     (stroke (width 0) (type default))
   )
-  (wire (pts (xy 166.37 46.99) (xy 166.37 48.26))
-    (stroke (width 0) (type default))
-  )
-  (text "LINE means supply connected After LVMS-> ASMS-> RES-> 2\nRequired by T15 2.2"
-    (at 171.45 58.42 0)
-    (effects (font (size 1.27 1.27) italic) (justify left bottom))
-  )
-  (hierarchical_label "VALVE_SUPPLY" (shape output) (at 201.93 97.79 0) (fields_autoplaced)
-    (effects (font (size 1.27 1.27)) (justify left))
-  )
   (hierarchical_label "SAFE_IN" (shape input) (at 156.21 59.69 90) (fields_autoplaced)
     (effects (font (size 1.27 1.27)) (justify left))
@@
         (path "/d921fbb5-521e-405d-bdec-f40195adfa1c/81567b80-5afb-49a2-8e1a-6e4e57e56b9d"
           (reference "D12") (unit 1)
-        )
-      )
-    )
-  )
-  (symbol (lib_id "power:PWR_FLAG") (at 156.21 45.72 0) (unit 1)
-    (in_bom yes) (on_board yes) (dnp no) (fields_autoplaced)
-    (property "Reference" "#FLG0101" (at 156.21 43.815 0)
-      (effects (font (size 1.27 1.27)) hide)
-    )
-    (property "Value" "PWR_FLAG" (at 156.21 40.64 0)
-      (effects (font (size 1.27 1.27)))
-    )
-    (property "Footprint" "" (at 156.21 45.72 0)
-      (effects (font (size 1.27 1.27)) hide)
-    )
-    (property "Datasheet" "~" (at 156.21 45.72 0)
-      (effects (font (size 1.27 1.27)) hide)
-    )
-    (pin "1")
-    (instances
-      (project "PUTM_DV_EBS_2023"
-        (path "/d921fbb5-521e-405d-bdec-f40195adfa1c/81567b80-5afb-49a2-8e1a-6e4e57e56b9d"
-          (reference "#FLG0101") (unit 1)
         )
       )
@@
         )
       )
-    )
-  )
-  (symbol (lib_id "power:LINE") (at 166.37 46.99 0) (unit 1)
-    (in_bom yes) (on_board yes) (dnp no) (fields_autoplaced)
-    (property "Reference" "#PWR0107" (at 166.37 50.8 0)
-      (effects (font (size 1.27 1.27)) hide)
-    )
-    (property "Value" "LINE" (at 166.37 41.91 0)
-      (effects (font (size 1.27 1.27)))
-    )
-    (property "Footprint" "" (at 166.37 46.99 0)
-      (effects (font (size 1.27 1.27)) hide)
-    )
-    (property "Datasheet" "" (at 166.37 46.99 0)
-      (effects (font (size 1.27 1.27)) hide)
-    )
-    (pin "1")
-    (instances
-      (project "PUTM_DV_EBS_2023"
-        (path "/d921fbb5-521e-405d-bdec-f40195adfa1c/81567b80-5afb-49a2-8e1a-6e4e57e56b9d"
-          (reference "#PWR0107") (unit 1)
-        )
-      )

Commit message: changed pcb version
Parts:
- D12: footprint Diode_SMD:D_SMA -> Diode_SMD:D_SMA_Handsoldering; symbol Diode:1N5817 -> Diode:1N5408
- R1: value 100R -> 1k
Connections:
- net VALVE_SUPPLY: now reaches K2.21
- net LINE: now reaches K2.24
- no-connect marks 4 -> 2
Other:
- note added: "LINE means supply connected After LVMS-> ASMS-> RES-> 2 Required by T15 2.2"
