File: hardware/sensors.kicad_sch (KiCad schematic)
At the start: 0 parts

Commit message: working simulations, assigned footprints
"nightly" relase
Other:
- added sheet Pressure Buffer (buffer.kicad_sch)
- added sheet Pressure Buffer1 (buffer.kicad_sch)
- added sheet Pressure Buffer2 (buffer.kicad_sch)
- note added: "10 bar 24V DC supply M5"
- note added: "PSE540-1W5"
Changed lines of the file:
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@@
 (kicad_sch (version 20211123) (generator eeschema)
   (paper "A4")
+  (wire (pts (xy 148.59 83.82) (xy 166.37 83.82))
+    (stroke (width 0) (type default) (color 0 0 0 0))
+  )
+  (wire (pts (xy 87.63 52.07) (xy 100.33 52.07))
+    (stroke (width 0) (type default) (color 0 0 0 0))
+  )
+  (wire (pts (xy 148.59 52.07) (xy 166.37 52.07))
+    (stroke (width 0) (type default) (color 0 0 0 0))
+  )
+  (wire (pts (xy 148.59 116.84) (xy 163.83 116.84))
+    (stroke (width 0) (type default) (color 0 0 0 0))
+  )
+  (wire (pts (xy 85.09 83.82) (xy 100.33 83.82))
+    (stroke (width 0) (type default) (color 0 0 0 0))
+  )
+  (wire (pts (xy 93.98 116.84) (xy 100.33 116.84))
+    (stroke (width 0) (type default) (color 0 0 0 0))
+  )
+  (text "10 bar 24V DC supply M5" (at 53.34 191.77 0)
+    (effects (font (size 6 6)) (justify left bottom))
+  )
+  (text "PSE540-1W5" (at 80.01 179.07 0)
+    (effects (font (size 6 6)) (justify left bottom))
+  )
+  (hierarchical_label "REDUNDANT" (shape output) (at 163.83 116.84 0)
+    (effects (font (size 1.27 1.27)) (justify left))
+  )
+  (hierarchical_label "MAIN" (shape output) (at 166.37 52.07 0)
+    (effects (font (size 1.27 1.27)) (justify left))
+  )
+  (hierarchical_label "SENSOR_REDUNDANT" (shape input) (at 93.98 116.84 180)
+    (effects (font (size 1.27 1.27)) (justify right))
+  )
+  (hierarchical_label "SENSOR_MAIN" (shape input) (at 87.63 52.07 180)
+    (effects (font (size 1.27 1.27)) (justify right))
+  )
+  (hierarchical_label "EBS" (shape output) (at 166.37 83.82 0)
+    (effects (font (size 1.27 1.27)) (justify left))
+  )
+  (hierarchical_label "SENSOR_EBS" (shape input) (at 85.09 83.82 180)
+    (effects (font (size 1.27 1.27)) (justify right))
+  )
+  (sheet (at 100.33 71.12) (size 48.26 24.13) (fields_autoplaced)
+    (stroke (width 0.1524) (type solid) (color 0 0 0 0))
+    (fill (color 0 0 0 0.0000))
+    (property "Sheet name" "Pressure Buffer1" (id 0) (at 100.33 70.4084 0)
+      (effects (font (size 1.27 1.27)) (justify left bottom))
+    )
+    (property "Sheet file" "buffer.kicad_sch" (id 1) (at 100.33 95.8346 0)
+      (effects (font (size 1.27 1.27)) (justify left top))
+    )
+    (pin "AIR_SENSOR" output (at 148.59 83.82 0)
+      (effects (font (size 1.27 1.27)) (justify right))
+    )
+    (pin "AIR_R" input (at 100.33 83.82 180)
+      (effects (font (size 1.27 1.27)) (justify left))
+    )
+  )
+  (sheet (at 100.33 39.37) (size 48.26 24.13) (fields_autoplaced)
+    (stroke (width 0.1524) (type solid) (color 0 0 0 0))
+    (fill (color 0 0 0 0.0000))
+    (property "Sheet name" "Pressure Buffer" (id 0) (at 100.33 38.6584 0)
+      (effects (font (size 1.27 1.27)) (justify left bottom))
+    )
+    (property "Sheet file" "buffer.kicad_sch" (id 1) (at 100.33 64.0846 0)
+      (effects (font (size 1.27 1.27)) (justify left top))
+    )
+    (pin "AIR_SENSOR" output (at 148.59 52.07 0)
+      (effects (font (size 1.27 1.27)) (justify right))
+    )
+    (pin "AIR_R" input (at 100.33 52.07 180)
+      (effects (font (size 1.27 1.27)) (justify left))
+    )
+  )
+  (sheet (at 100.33 102.87) (size 48.26 24.13) (fields_autoplaced)
+    (stroke (width 0.1524) (type solid) (color 0 0 0 0))
+    (fill (color 0 0 0 0.0000))
+    (property "Sheet name" "Pressure Buffer2" (id 0) (at 100.33 102.1584 0)
+      (effects (font (size 1.27 1.27)) (justify left bottom))
+    )
+    (property "Sheet file" "buffer.kicad_sch" (id 1) (at 100.33 127.5846 0)
+      (effects (font (size 1.27 1.27)) (justify left top))
+    )
+    (pin "AIR_SENSOR" output (at 148.59 116.84 0)
+      (effects (font (size 1.27 1.27)) (justify right))
+    )
+    (pin "AIR_R" input (at 100.33 116.84 180)
+      (effects (font (size 1.27 1.27)) (justify left))
+    )
+  )
 )
